File: hardware/motors/motors.kicad_sch (KiCad schematic)
At the start: 26 parts, among them J1 24V, J2 12V, J3 Motor1, J4 Motor2, J5 Conn_01x03_Pin, Q1 IRF540N, Q2 IRF540N, U1 4N25, U2 LM317_TO-220, U3 4N25

Commit message: Adicionando perfil de amendoim
Parts:
- R1, R7: value 470R -> 220R
